File: hw/solitaire/solitaire.kicad_pcb (KiCad board)
At the start: 2 copper layers, 100 x 60 mm, 16 parts, among them J1 51441-1093, J2 SKQUCAA010, J3 SBW, J4 BATT_IN, SW1 DEAL, SW2 UNDO, U1 TPS63900, U2 MSP430FR2355TDBTR

Commit message: Rename nav switch J2->SW3, add direction net labels, document case dimensions
Renamed the SKQUCAA010 nav switch reference from J2 (Ultra Librarian's
default connector prefix) to SW3 to match the SW1/SW2 naming convention,
and added NAV_UP/DOWN/LEFT/RIGHT/CENTER net labels on its schematic pins
so the up/down/left/right mapping is legible without cross-referencing
the datasheet.

Also adds docs/case_design_dimensions.md: verified component positions
and mechanical envelopes pulled from datasheets for FreeCAD case design,
including nav switch stem geometry/pivot point for sizing a knob cutout
and the selected 2xAA battery holder (Adafruit #4194).

Co-Authored-By: Claude Sonnet 5 <noreply@anthropic.com>
Parts:
- renumbered J2 to SW3
Changed lines of the file:
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@@
 		(at 74.1 74.33)
 		(tags "SKQUCAA010 ")
-		(property "Reference" "J2"
+		(property "Reference" "SW3"
 			(at 4.15305 -3.33 0)
 			(unlocked yes)

Commit message: Replace obsolete Molex 51441-1093 with GCT FFC2B35-10-T at J1
Molex 51441-1093 (display FPC connector) is EOL/no longer manufactured.
Registers GCT FFC2B35-10-T's symbol/footprint library and swaps J1 over
on both the schematic and PCB, preserving the existing pin-to-signal
mapping (already verified against the Sharp LS013B7DH03's real terminal
numbers) and the existing net assignments.

The new symbol's pin layout differs from the old one (single column vs
two columns of 6), which required adding wiring for pins 6-10 and two
extra pins (11/12, the connector's mechanical/shield pads) that GCT's
stock symbol doesn't expose but the old design tied to GND. PCB footprint
replaced with GCT's real pad geometry at the same position/rotation;
render-verified the cable-entry edge still faces the LCD outline.

Documents the swap and the underlying obsolescence research in
docs/case_design_dimensions.md.

Co-Authored-By: Claude Sonnet 5 <noreply@anthropic.com>
Parts:
- J1: value 51441-1093 -> FFC2B35-10-T; footprint 514411093:CON10_1X10_DRB_51441_MOL -> FFC2B35_10_T:CONN_FFC2B35-10-x_GCT
Changed lines of the file:
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@@
 		)
 	)
-	(footprint "514411093:CON10_1X10_DRB_51441_MOL"
+	(footprint "FFC2B35_10_T:CONN_FFC2B35-10-x_GCT"
 		(layer "F.Cu")
 		(at 94.77 77.5 90)
-		(tags "514411093 ")
+		(tags "FFC2B35-10-T ")
 		(property "Reference" "J1"
 			(at 0 -3.77 90)
@@
 			)
 		)
-		(property "Value" "51441-1093"
+		(property "Value" "FFC2B35-10-T"
 			(at 5.5 0.23 0)
 			(unlocked yes)
@@
 			)
 		)
-		(property "Datasheet" "514411093"
+		(property "Datasheet" "FFC2B35-10-T"
 			(at 0 0 90)
 			(layer "F.Fab")
@@
 			)
 		)
-		(property "Description" "Molex 51441-1093, 10-position 0.5mm pitch bottom-contact FPC/FFC connector"
+		(property "Description" "GCT FFC2B35-10-T, 10-position 0.5mm pitch bottom-contact front-flip FPC/FFC connector - replacement for obsolete Molex 51441-1093"
 			(at 0 0 90)
 			(layer "F.Fab")
@@
 			)
 		)
-		(property ki_fp_filters "CON10_1X10_DRB_51441_MOL")
+		(property ki_fp_filters "CONN_FFC2B35-10-x_GCT")
 		(sheetname "/")
 		(sheetfile "solitaire.kicad_sch")
 		(attr smd)
 		(fp_line
-			(start 3.7719 -2.2352)
-			(end -3.7719 -2.2352)
-			(stroke
-				(width 0.1524)
-				(type solid)
-			)
-			(layer "F.SilkS")
-		)
-		(fp_line
-			(start -3.7719 -2.2352)
-			(end -3.7719 -2.02184)
-			(stroke
-				(width 0.1524)
-				(type solid)
-			)
-			(layer "F.SilkS")
-		)
-		(fp_line
-			(start 3.7719 -2.02184)
-			(end 3.7719 -2.2352)
-			(stroke
-				(width 0.1524)
-				(type solid)
-			)
-			(layer "F.SilkS")
-		)
-		(fp_line
-			(start -3.7719 0.14224)
-			(end -3.7719 1.2192)
-			(stroke
-				(width 0.1524)
-				(type solid)
-			)
-			(layer "F.SilkS")
-		)
-		(fp_line
-			(start 3.7719 1.2192)
-			(end 3.7719 0.14224)
-			(stroke
-				(width 0.1524)
-				(type solid)
-			)
-			(layer "F.SilkS")
-		)
-		(fp_line
-			(start 2.73124 1.2192)
-			(end 3.7719 1.2192)
-			(stroke
-				(width 0.1524)
-				(type solid)
-			)
-			(layer "F.SilkS")
-		)
-		(fp_line
-			(start -3.7719 1.2192)
-			(end -2.73124 1.2192)
-			(stroke
-				(width 0.1524)
-				(type solid)
-			)
-			(layer "F.SilkS")
-		)
-		(fp_line
-			(start 4.1021 -2.3622)
-			(end -4.1021 -2.3622)
-			(stroke
-				(width 0.1524)
-				(type solid)
-			)
-			(layer "F.CrtYd")
-		)
-		(fp_line
-			(start -4.1021 -2.3622)
-			(end -4.1021 2.1844)
-			(stroke
-				(width 0.1524)
-				(type solid)
-			)
-			(layer "F.CrtYd")
-		)
-		(fp_line
-			(start 4.1021 2.1844)
-			(end 4.1021 -2.3622)
-			(stroke
-				(width 0.1524)
-				(type solid)
-			)
-			(layer "F.CrtYd")
-		)
-		(fp_line
-			(start -4.1021 2.1844)
-			(end 4.1021 2.1844)
-			(stroke
-				(width 0.1524)
-				(type solid)
-			)
-			(layer "F.CrtYd")
-		)
-		(fp_line
-			(start 3.6449 -2.1082)
-			(end -3.6449 -2.1082)
-			(stroke
-				(width 0.0254)
-				(type solid)
-			)
-			(layer "F.Fab")
-		)
-		(fp_line
-			(start -3.6449 -2.1082)
-			(end -3.6449 1.0922)
-			(stroke
-				(width 0.0254)
-				(type solid)
-			)
-			(layer "F.Fab")
-		)
-		(fp_line
-			(start 3.6449 1.0922)
-			(end 3.6449 -2.1082)
-			(stroke
-				(width 0.0254)
-				(type solid)
-			)
-			(layer "F.Fab")
-		)
-		(fp_line
-			(start 2.885 1.0922)
-			(end 2.25 2.3622)
-			(stroke
-				(width 0.0254)
-				(type solid)
-			)
-			(layer "F.Fab")
-		)
-		(fp_line
-			(start 1.615 1.0922)
-			(end 2.25 2.3622)
-			(stroke
-				(width 0.0254)
-				(type solid)
-			)
-			(layer "F.Fab")
-		)
-		(fp_line
-			(start -3.6449 1.0922)
-			(end 3.6449 1.0922)
-			(stroke
-				(width 0.0254)
-				(type solid)
-			)
-			(layer "F.Fab")
-		)
-		(fp_text user "${REFERENCE}"
-			(at 0 1.6002 90)
-			(unlocked yes)
-			(layer "F.Fab")
-			(effects
-				(font
-					(size 1 1)
-					(thickness 0.15)
-				)
-			)
+			(start -5.305699 -4.474299)
+			(end -5.305699 3.2766)
+			(stroke
+				(width 0.1524)
+				(type solid)
+			)
+			(layer "F.CrtYd")
+		)
+		(fp_line
+			(start -5.305699 3.2766)
+			(end 5.305699 3.2766)
+			(stroke
+				(width 0.1524)
+				(type solid)
+			)
+			(layer "F.CrtYd")
+		)
+		(fp_line
+			(start 5.305699 3.2766)
+			(end 5.305699 -4.474299)
+			(stroke
+				(width 0.1524)
+				(type solid)
+			)
+			(layer "F.CrtYd")
+		)
+		(fp_line
+			(start 5.305699 -4.474299)
+			(end -5.305699 -4.474299)
+			(stroke
+				(width 0.1524)
+				(type solid)
+			)
+			(layer "F.CrtYd")
+		)
+		(fp_circle
+			(center -2.25 -5.477599)
+			(end -1.869 -5.477599)
+			(stroke
+				(width 0.508)
+				(type solid)
+			)
+			(fill none)
+			(layer "F.Fab")
+		)
+		(fp_circle
+			(center -6.604 -3.572599)
+			(end -6.223 -3.572599)
+			(stroke
+				(width 0.508)
+				(type solid)
+			)
+			(fill none)
+			(layer "F.SilkS")
+		)
+		(fp_line
+			(start -4.826 3.1496)
+			(end 4.826 3.1496)
+			(stroke
+				(width 0.1524)
+				(type solid)
+			)
+			(layer "F.SilkS")
+		)
+		(fp_line
+			(start 4.826 3.1496)
+			(end 4.826 1.115042)
+			(stroke
+				(width 0.1524)
+				(type solid)
+			)
+			(layer "F.SilkS")
+		)
+		(fp_line
+			(start 4.826 -3.149599)
+			(end 2.735141 -3.149599)
+			(stroke
+				(width 0.1524)
+				(type solid)
+			)
+			(layer "F.SilkS")
+		)
+		(fp_line
+			(start -4.826 -3.149599)
+			(end -4.826 -1.760238)
+			(stroke
+				(width 0.1524)
+				(type solid)
+			)
+			(layer "F.SilkS")
 		)
 		(pad "1" smd rect
-			(at 2.250001 1.6002 90)
-			(size 0.3048 0.6604)
+			(at -2.250001 -3.572599)
+			(size 0.3048 1.2954)
 			(layers "F.Cu" "F.Mask" "F.Paste")
 			(net 41 "Net-(U2-P4.5_UCB1CLK)")
@@
 		)
 		(pad "2" smd rect
-			(at 1.749999 1.6002 90)
-			(size 0.3048 0.6604)
+			(at -1.749999 -3.572599)
+			(size 0.3048 1.2954)
 			(layers "F.Cu" "F.Mask" "F.Paste")
 			(net 42 "Net-(U2-P4.6_UCB1SIMO_UCB1SDA)")
@@
 		)
 		(pad "3" smd rect
-			(at 1.25 1.6002 90)
-			(size 0.3048 0.6604)
+			(at -1.25 -3.572599)
+			(size 0.3048 1.2954)
 			(layers "F.Cu" "F.Mask" "F.Paste")
 			(net 43 "Net-(U2-P4.4_UCB1STE)")
@@
 		)
 		(pad "4" smd rect
-			(at 0.750001 1.6002 90)
-			(size 0.3048 0.6604)
+			(at -0.750001 -3.572599)
+			(size 0.3048 1.2954)
 			(layers "F.Cu" "F.Mask" "F.Paste")
 			(net 2 "Net-(U2-P5.0_TB2.1_MFM.RX_A8)")
@@
 		)
 		(pad "5" smd rect
-			(at 0.25 1.6002 90)
-			(size 0.3048 0.6604)
+			(at -0.25 -3.572599)
+			(size 0.3048 1.2954)
 			(layers "F.Cu" "F.Mask" "F.Paste")
 			(net 40 "Net-(U2-P5.1_TB2.2_MFM.TX_A9)")
@@
 		)
 		(pad "6" smd rect
-			(at -0.25 1.6002 90)
-			(size 0.3048 0.6604)
+			(at 0.25 -3.572599)
+			(size 0.3048 1.2954)
 			(layers "F.Cu" "F.Mask" "F.Paste")
 			(net 26 "VCC")
@@
 		)
 		(pad "7" smd rect
-			(at -0.750001 1.6002 90)
-			(size 0.3048 0.6604)
+			(at 0.750001 -3.572599)
+			(size 0.3048 1.2954)
 			(layers "F.Cu" "F.Mask" "F.Paste")
 			(net 26 "VCC")
@@
 		)
 		(pad "8" smd rect
-			(at -1.25 1.6002 90)
-			(size 0.3048 0.6604)
+			(at 1.25 -3.572599)
+			(size 0.3048 1.2954)
 			(layers "F.Cu" "F.Mask" "F.Paste")
 			(net 26 "VCC")
@@
 		)
 		(pad "9" smd rect
-			(at -1.749999 1.6002 90)
-			(size 0.3048 0.6604)
+			(at 1.749999 -3.572599)
+			(size 0.3048 1.2954)
 			(layers "F.Cu" "F.Mask" "F.Paste")
 			(net 1 "GND")
@@
 		)
 		(pad "10" smd rect
-			(at -2.250001 1.6002 90)
-			(size 0.3048 0.6604)
+			(at 2.250001 -3.572599)
+			(size 0.3048 1.2954)
 			(layers "F.Cu" "F.Mask" "F.Paste")
 			(net 1 "GND")
@@
 		)
 		(pad "11" smd rect
-			(at -3.4163 -0.9398 90)
-			(size 0.8636 1.4986)
+			(at -4.149999 -0.322598)
+			(size 1.8034 2.2098)
 			(layers "F.Cu" "F.Mask" "F.Paste")
 			(net 1 "GND")
@@
 		)
 		(pad "12" smd rect
-			(at 3.4163 -0.9398 90)
-			(size 0.8636 1.4986)
-			(layers "F.Cu" "F.Mask" "F.Paste")
-			(net 1 "GND")
+			(at 4.149999 -0.322598)
+			(size 1.8034 2.2098)
+			(layers "F.Cu" "F.Mask" "F.Paste")
+			(net 1 "GND")
