File: hw/solitaire/solitaire.kicad_pcb (KiCad board)
At the start: 2 copper layers, 100 x 60 mm, 16 parts, among them J1 51441-1093, J3 SBW, J4 BATT_IN, SW1 DEAL, SW2 UNDO, SW3 SKQUCAA010, U1 TPS63900, U2 MSP430FR2355TDBTR

Commit message: Re-swap J1 to GCT FFC2B35-10-T, fill GND plane, fix DRC/ERC violations
Redoes the obsolete-Molex-to-GCT J1 connector swap (previously reverted
in bc0f137) with fresh EDA files from JLCPCB, and ties up the loose ends
that were left dangling mid-edit:

- J1 pins 11/12 (mechanical/shield pads) were floating with no net,
  sitting directly on GND copper - added the pins to the FFC2B35-10-T
  symbol (embedded copy + external .kicad_sym), wired them to a new
  GND flag, and set the matching PCB pads to the GND net. Fixes 2
  shorting_items, 1 clearance, 1 hole_clearance, and 4 solder_mask_bridge
  DRC violations.
- The B.Cu GND zone existed but had never been filled, fragmenting the
  ground net into disconnected islands. Filled it, resolving 12 dangling
  vias and 12 missing-connection DRC warnings.
- J1's silkscreen reference was clipped by its own solder mask - moved
  it below the connector body.

kicad-cli pcb drc: 23 violations + 12 unconnected -> 0/0.
kicad-cli sch erc: same 31-warning baseline plus the expected
"unspecified pintype" nags for the 2 new pins - no new genuine errors.

Co-Authored-By: Claude Sonnet 5 <noreply@anthropic.com>
Parts:
- C3: value 1 uf -> 1uF
- J1: value 51441-1093 -> FFC2B35-10-T; footprint 514411093:CON10_1X10_DRB_51441_MOL -> disp:CONN_FFC2B35-10-x_GCT
Connections:
- net Net-(U2-P3.0_MCLK) renamed /NAV_CENTER
- net Net-(U2-P3.1_OA2O) renamed /NAV_RIGHT
- net Net-(U2-P3.3_OA2+) renamed /NAV_UP
- net Net-(U2-P3.4_SMCLK) renamed /NAV_LEFT
- net Net-(U2-P3.5_OA3O) renamed /NAV_DOWN
- net Net-(U2-P4.4_UCB1STE) renamed /SCS
- net Net-(U2-P4.5_UCB1CLK) renamed /SCLK
- net Net-(U2-P4.6_UCB1SIMO_UCB1SDA) renamed /SI
- net Net-(U2-P5.0_TB2.1_MFM.RX_A8) renamed /SCOM
- net Net-(U2-P5.1_TB2.2_MFM.TX_A9) renamed /DISP
Routing:
- net /SCLK: track 62.1 -> 44.4 mm
- net /SCS: track 58.1 -> 49.4 mm
- net /SI: track 54.7 -> 46.7 mm
- net VCC: track 137.8 -> 145.4 mm
- net /DISP: track 54.1 -> 61.0 mm, vias 2 -> 3
- net Net-(J3-Pin_2): track 36.7 -> 35.6 mm
- net GND: track 61.1 -> 62.0 mm
- net /SCOM: track 45.9 -> 45.1 mm

Commit message: Add 4 M2.5 mounting holes to the PCB
Board had zero mounting holes, blocking case-boss placement (open item
#1 in case_design_dimensions.md). Added 4x MountingHole_2.7mm_M2.5
(NPTH, no copper) sized for M2.5 self-tapping screws into the FDM case
bosses.

True corners weren't all available - J3 blocks top-left flush with the
board edge, and the L1/U1/C1/C2/R1/R2 cluster blocks bottom-left - so
H3/H4 are shifted into the nearest clear pockets instead of sitting at
literal corners. H1/H2 landed at the (fully clear) top-right/bottom-right.

Refilled the B.Cu GND zone afterward since the new NPTH holes didn't
exist yet at the last fill and DRC flagged 0mm hole clearance against
the zone copper. DRC clean (0/0) after the refill.

Doc updated with the board-relative hole coordinates for the FreeCAD
case bosses.

Co-Authored-By: Claude Sonnet 5 <noreply@anthropic.com>
Parts:
- added H1: MountingHole_2.7mm_M2.5, MountingHole_2.7mm_M2.5, F.Cu at (135.0, 55.0)
- added H2: MountingHole_2.7mm_M2.5, MountingHole_2.7mm_M2.5, F.Cu at (135.0, 100.0)
- added H3: MountingHole_2.7mm_M2.5, MountingHole_2.7mm_M2.5, F.Cu at (55.0, 68.0)
- added H4: MountingHole_2.7mm_M2.5, MountingHole_2.7mm_M2.5, F.Cu at (69.0, 101.0)
